Commit message: ver2.2 增加了获得相对位置的接口

File: Webots_PR2_Path_Planning/protos/urdf_arm_mix/urdf/urdf_arm_mix.urdf (robot description, URDF)
Before this commit: robot urdf_arm, 50 links, 49 joints
Links:
- added link left_intermediate_link, mass 0.1; collision box size=0.05 0.05 0.02; visual box size=0.05 0.05 0.02
- added link right_intermediate_link, mass 0.1; collision box size=0.05 0.05 0.02; visual box size=0.05 0.05 0.02
Joints:
- added joint left_intermediate_joint: type revolute, parent zarm_l5_link, child left_intermediate_link, origin xyz=0 0 -0.1 rpy=0 0 0, axis 1 0 0, limit lower=-1.57 upper=1.57 effort=10.0 velocity=5.0
- added joint right_intermediate_joint: type revolute, parent zarm_r5_link, child right_intermediate_link, origin xyz=0 0 -0.1 rpy=0 0 0, axis 1 0 0, limit lower=-1.57 upper=1.57 effort=10.0 velocity=5.0
- joint left_gripper_attachment_joint: origin xyz=0 0 -0.1 rpy=3.14 0 0 -> xyz=0 0 0 rpy=3.14 0 0; parent zarm_l5_link -> left_intermediate_link
- joint right_gripper_attachment_joint: origin xyz=0 0 -0.1 rpy=3.14 0 0 -> xyz=0 0 0 rpy=3.14 0 0; parent zarm_r5_link -> right_intermediate_link
